File: EWB node/blt.sch (KiCad schematic (older format))
At the start: 3 parts, among them Q1 DMN6140L

Commit message: pcb layout
Changed lines of the file:
@@
 $Descr A4 11693 8268
 encoding utf-8
-Sheet 2 12
+Sheet 10 12
 Title ""
 Date ""
@@
 AR Path="/61376E8C/6116AB3D" Ref="Q14"  Part="1"
 AR Path="/613824D3/6116AB3D" Ref="Q15"  Part="1"
-F 0 "Q1" V 5499 4750 50  0000 C CNN
+F 0 "Q13" V 5499 4750 50  0000 C CNN
 F 1 "DMN6140L" V 5590 4750 50  0000 C CNN
 F 2 "Package_TO_SOT_SMD:SOT-23" H 5450 4675 50  0001 L CIN
@@
 AR Path="/61376E8C/61170761" Ref="#PWR058"  Part="1"
 AR Path="/613824D3/61170761" Ref="#PWR060"  Part="1"
-F 0 "#PWR032" H 5500 4150 50  0001 C CNN
+F 0 "#PWR056" H 5500 4150 50  0001 C CNN
 F 1 "+3.3V" H 5515 4473 50  0000 C CNN
 F 2 "" H 5500 4300 50  0001 C CNN
@@
 AR Path="/61376E8C/6117136D" Ref="#PWR057"  Part="1"
 AR Path="/613824D3/6117136D" Ref="#PWR059"  Part="1"
-F 0 "#PWR031" H 4800 4200 50  0001 C CNN
+F 0 "#PWR055" H 4800 4200 50  0001 C CNN
 F 1 "+5V" H 4815 4523 50  0000 C CNN
 F 2 "" H 4800 4350 50  0001 C CNN
@@
 AR Path="/61376E8C/6116A503" Ref="R31"  Part="1"
 AR Path="/613824D3/6116A503" Ref="R33"  Part="1"
-F 0 "R5" H 4870 4646 50  0000 L CNN
+F 0 "R29" H 4870 4646 50  0000 L CNN
 F 1 "10k" H 4870 4555 50  0000 L CNN
 F 2 "Resistor_SMD:R_0603_1608Metric_Pad0.98x0.95mm_HandSolder" V 4730 4600 50  0001 C CNN
@@
 AR Path="/61376E8C/6116EB86" Ref="R32"  Part="1"
 AR Path="/613824D3/6116EB86" Ref="R34"  Part="1"
-F 0 "R6" H 5720 4646 50  0000 L CNN
+F 0 "R30" H 5720 4646 50  0000 L CNN
 F 1 "10k" H 5720 4555 50  0000 L CNN
 F 2 "Resistor_SMD:R_0603_1608Metric_Pad0.98x0.95mm_HandSolder" V 5580 4600 50  0001 C CNN
